File: documentation/circuits/introduction/introduction.sch (KiCad schematic (older format))
At the start: 0 parts

Commit message: update
Parts:
- added U?: 7404, symbol dismpy:7404
- added U?: 7408, symbol dismpy:7408
- added U? (x9): 7400, symbol dismpy:7400
Connections:
- net labels added: output
- net labels removed: result
- wire segments 4 -> 53
